Commit message: update

File: st_gazebo/urdf/robot1.urdf (robot description, URDF)
Before this commit: robot robot1, 3 links, 2 joints
Links:
- added link arm1; visual box size=0.2 0.04 0.02
- added link arm2; visual box size=0.2 0.04 0.02
- added link arm3; visual box size=0.1 0.04 0.02
- added link arm_base; visual box size=0.05 0.05 0.1
- added link left_camera; visual box size=0.1 0.02 0.01
- link body_link: geometry visual box size=0.6 0.4 0.2
- link elevator: mass 1 -> None; geometry visual box size=0.1 0.4 0.02
Joints:
- added joint arm1_joint: type revolute, parent arm_base, child arm1, origin xyz=0 0 0.06, axis 0 0 1, limit lower=-15 upper=15 effort=1000.0 velocity=30
- added joint arm2_joint: type revolute, parent arm1, child arm2, origin xyz=0.2 0 -0.02, axis 0 0 1, limit lower=-15 upper=15 effort=1000.0 velocity=30
- added joint arm3_joint: type revolute, parent arm2, child arm3, origin xyz=0.2 0 -0.02, axis 0 0 1, limit lower=-15 upper=15 effort=1000.0 velocity=30
- added joint arm_base_joint: type fixed, parent elevator, child arm_base, origin xyz=0.05 0 0.05 rpy=0 0 3.1415
- added joint left_camera_joint: type fixed, parent elevator, child left_camera, origin xyz=-0.1 0.05 0.2 rpy=-1.8326 0 0
- joint body_joint: origin xyz=0.5 0 0 rpy=0 0 0 -> xyz=-0.15 0 0.2 rpy=0 0 0
- joint elevator_joint: axis 1 0 0 -> 0 0 1; origin xyz=0.0 0.0 0.0 -> xyz=0.1 0 0.45
